File: 12vBatteryPack/BatteryPack.kicad_pcb (KiCad board)
At the start: 2 copper layers, 80 x 153.7 mm, 14 parts, among them J1 Conn_01x02_Male, J2 Conn_01x07_Male, J3 Conn_01x02_Male

Commit message: Added untracked projects
Parts:
- removed BT4, BT5, BT6: Battery_Cell, Battery:BatteryHolder_MPD_BH-18650-PC2
- removed J2: Conn_01x07_Male, BatteryPack:SolderWire-0.5sqmm_1x07_P4.8mm_D0.9mm_OD2.3mm
- moved BT2 64.5 mm to (44.5, 119.9)
- moved BT3 64.5 mm to (44.5, 140.2)
- moved BT1 64.5 mm to (44.5, 99.6)
Connections:
- BT3 pad 1: BAT_BAL3 -> BAT+
Routing:
- net BAT+: track 127.5 -> 0.00 mm
- net BAT_BAL5: track 115.0 -> 0.00 mm
- net BAT_BAL4: track 101.9 -> 0.00 mm
- net BAT_BAL3: track 84.9 -> 0.00 mm
- net BAT_BAL2: track 71.2 -> 0.00 mm
- net BAT_BAL1: track 69.6 -> 0.00 mm
- removed copper zone on F.Cu, net BAT_BAL1
- removed copper zone on F.Cu, net BAT_BAL2
- removed copper zone on F.Cu, net BAT_BAL3
