File: ATTinyCard/ATTinyCard.kicad_sch (KiCad schematic)
At the start: 1 part

Commit message: Added untracked projects
Parts:
- added J1: Conn_01x01_Female, Connector_PinHeader_2.54mm:PinHeader_1x01_P2.54mm_Horizontal, symbol Connector:Conn_01x01_Female
- U1: renamed from U?; footprint Package_DIP:DIP-8_W7.62mm -> EmbeddedParts:DIP8-Embedded
Connections:
- net at U1.8 (VCC): now also J1.1 (Pin_1)
Changed lines of the file:
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@@
 (kicad_sch (version 20211123) (generator eeschema)
   (paper "A4")
+  (wire (pts (xy 107.95 69.85) (xy 109.22 69.85))
+    (stroke (width 0) (type default) (color 0 0 0 0))
+  )
+  (wire (pts (xy 107.95 80.01) (xy 107.95 69.85))
+    (stroke (width 0) (type default) (color 0 0 0 0))
+  )
   (symbol (lib_id "MCU_Microchip_ATtiny:ATtiny85-20P") (at 107.95 95.25 0) (unit 1)
     (in_bom yes) (on_board yes) (fields_autoplaced)
-    (property "Reference" "U?" (id 0) (at 94.488 94.3415 0)
+    (property "Reference" "U1" (id 0) (at 94.488 94.3415 0)
       (effects (font (size 1.27 1.27)) (justify right))
     )
@@
       (effects (font (size 1.27 1.27)) (justify right))
     )
-    (property "Footprint" "Package_DIP:DIP-8_W7.62mm" (id 2) (at 107.95 95.25 0)
+    (property "Footprint" "EmbeddedParts:DIP8-Embedded" (id 2) (at 107.95 95.25 0)
       (effects (font (size 1.27 1.27) italic) hide)
     )
@@
     (pin "8")
   )
+  (symbol (lib_id "Connector:Conn_01x01_Female") (at 114.3 69.85 0) (unit 1)
+    (in_bom yes) (on_board yes) (fields_autoplaced)
+    (property "Reference" "J1" (id 0) (at 115.0112 68.9415 0)
+      (effects (font (size 1.27 1.27)) (justify left))
+    )
+    (property "Value" "Conn_01x01_Female" (id 1) (at 115.0112 71.7166 0)
+      (effects (font (size 1.27 1.27)) (justify left))
+    )
+    (property "Footprint" "Connector_PinHeader_2.54mm:PinHeader_1x01_P2.54mm_Horizontal" (id 2) (at 114.3 69.85 0)
+      (effects (font (size 1.27 1.27)) hide)
+    )
+    (property "Datasheet" "~" (id 3) (at 114.3 69.85 0)
+      (effects (font (size 1.27 1.27)) hide)
+    )
+    (pin "1")
+  )
   (sheet_instances
     (path "/" (page "1"))
   )
   (symbol_instances
+    (path "/f888d71b-37ae-40d1-b9f5-0cb7096abe99"
+      (reference "J1") (unit 1) (value "Conn_01x01_Female") (footprint "Connector_PinHeader_2.54mm:PinHeader_1x01_P2.54mm_Horizontal")
+    )
     (path "/3eb6166e-d2a4-4778-a9e3-fd9ea19f972e"
-      (reference "U?") (unit 1) (value "ATtiny85-20P") (footprint "Package_DIP:DIP-8_W7.62mm")
+      (reference "U1") (unit 1) (value "ATtiny85-20P") (footprint "EmbeddedParts:DIP8-Embedded")
     )
   )
