File: TheSun2/TheSun2.sch (KiCad schematic (older format))
At the start: 7 parts, among them J1 Conn_02x20_Odd_Even, J2 Conn_01x06_Male, J3 Conn_01x06_Male, J4 Screw_Terminal_01x02, J5 Screw_Terminal_01x02, Q1 IRLZ44N, Q2 IRLZ44N

Commit message: Added fancy pi power mosfet hat
Parts:
- removed J2, J3: Conn_01x06_Male, Connector_PinSocket_2.54mm:PinSocket_1x06_P2.54mm_Vertical, symbol Connector:Conn_01x06_Male
- removed J5: Screw_Terminal_01x02, TerminalBlock_Phoenix:TerminalBlock_Phoenix_MKDS-1,5-2-5.08_1x02_P5.08mm_Horizontal, symbol Connector:Screw_Terminal_01x02
- added D1, D2, D3, D4: LED, LED_SMD:LED_1206_3216Metric, symbol Device:LED_Small
- added J2, J3, J4: Screw_Terminal_01x02, TerminalBlock_4Ucon:TerminalBlock_4Ucon_1x02_P3.50mm_Horizontal, symbol Connector:Screw_Terminal_01x02
- added Q3, Q4: IRLR7843, Package_TO_SOT_SMD:TO-252-3_TabPin2, symbol Transistor_FET:IRLZ44N
- added R1, R10, R12, R3, R4, R6, R7, R9: 10K, Resistor_SMD:R_1206_3216Metric, symbol Device:R
- added R11, R2, R5, R8: 500R, Resistor_SMD:R_1206_3216Metric, symbol Device:R_Small
- added U1, U2, U3, U4, U5, U6, U7, U8: 2N7002H, Package_TO_SOT_SMD:SOT-23, symbol Transistor_FET:2N7002H
- J4: footprint TerminalBlock_Phoenix:TerminalBlock_Phoenix_MKDS-1,5-2-5.08_1x02_P5.08mm_Horizontal -> TerminalBlock_4Ucon:TerminalBlock_4Ucon_1x02_P3.50mm_Horizontal
- Q1, Q2: value IRLZ44N -> IRLR7843; footprint Package_TO_SOT_THT:TO-220-3_Vertical -> Package_TO_SOT_SMD:TO-252-3_TabPin2
Connections:
- net labels added: 3.3v, 5v, GND, GPIO-29, GPIO-31, PWM-32, PWM-33
- wire segments 40 -> 86
Other:
- moved on the sheet: J1, Q1
