File: TheSun3/TheSun2.kicad_pcb (KiCad board)
At the start: 2 copper layers, 114 x 92 mm, 62 parts, among them J1 Conn_01x02_Male, J10 Conn_01x06, J2 Conn_01x02_Male, J3 Conn_01x02_Male, J4 Conn_01x02, J5 Conn_01x02_Male, J6 Conn_01x02_Male, J7 Conn_01x02_Male, J8 Conn_01x02_Male, J9 Conn_01x02_Male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

Commit message: Added fancy pi power mosfet hat
Other:
- net class Default removed
- net class test removed
